Commit message: add gazebo

File: src/toybox_description/description/robot.urdf.xacro (robot description, xacro)
@@ -2,3 +2,4 @@
 <robot xmlns:xacro="http://www.ros.org/wiki/xacro" name="robot">
     <xacro:include filename="robot_core.xacro"/>
+    <xacro:include filename="gazebo_control.xacro"/>
 </robot>

File: src/toybox_description/description/robot_core.xacro (robot description, xacro)
@@ -28,4 +28,9 @@
         </xacro:inertial_box>
     </link>
+    <gazebo reference='chassis'>
+        <material>
+            Gazebo/white
+        </material>
+    </gazebo>
     <joint name="left_wheel_joint" type="continuous">
         <parent link="base_link"/>
@@ -50,4 +55,9 @@
         </xacro:inertial_cylinder>
     </link>
+    <gazebo reference='left_wheel'>
+        <material>
+            Gazebo/Blue
+        </material>
+    </gazebo>
     <joint name="right_wheel_joint" type="continuous">
         <parent link="base_link"/>
@@ -72,4 +82,9 @@
         </xacro:inertial_cylinder>
     </link>
+    <gazebo reference='right_wheel'>
+        <material>
+            Gazebo/Blue
+        </material>
+    </gazebo>
     <joint name="caster_wheel_joint" type="fixed">
         <parent link="chassis"/>
@@ -93,3 +108,8 @@
         </xacro:inertial_sphere>
     </link>
+    <gazebo reference='caster_wheel'>
+        <material>
+            Gazebo/white
+        </material>
+    </gazebo>
 </robot>
