Commit message: add depth camera

File: src/toybox_description/description/lidar.xacro (robot description, xacro)
@@ -4,5 +4,5 @@
         <parent link="base_link"/>
         <child link="laser_frame"/>
-        <origin xyz="0.13 0.0 0.09" rpy="0.0 0.0 0.0"/>
+        <origin xyz="0.13 0.0 0.085" rpy="0.0 0.0 0.0"/>
     </joint>
     <link name="laser_frame">
@@ -30,5 +30,5 @@
         <sensor name="laser" type="ray">
         <pose> 0 0 0 0 0 0 </pose>
-        <visualize>true</visualize>
+        <visualize>false</visualize>
         <update_rate>10</update_rate>
         <ray>

File: src/toybox_description/description/robot.urdf.xacro (robot description, xacro)
@@ -4,3 +4,4 @@
     <xacro:include filename="ros2_control.xacro"/>
     <xacro:include filename="lidar.xacro"/>
+    <xacro:include filename="depth_camera.xacro"/>
 </robot>
